Commit message: adding models for Ruby 80

File: src/vehicle/mr1000/urdf/mr1000_motor.urdf.xacro (robot description, xacro)
@@ -38,4 +38,5 @@
   <xacro:include filename="$(find mr1000)/urdf/VLP-64.urdf.xacro"/>
   <!-- <xacro:include filename="$(find velodyne_description)/urdf/RS-Ruby80.urdf.xacro"/> -->
+  <xacro:include filename="$(find mr1000)/urdf/Customized.urdf.xacro"/>
   <!-- <xacro:include filename="$(find velodyne_description)/urdf/VLP-16.urdf.xacro"/> -->
   <!-- Base link is the center of the robot's base -->
@@ -156,7 +157,11 @@
   </VLP-16> -->
   <!-- VLP-64 -->
-  <VLP-64 parent="base_link" name="sensor" topic="/sensor_scan" hz="10" samples="1800" gpu="${gpu}" >
+  <!-- <VLP-64 parent="base_link" name="sensor" topic="/sensor_scan" hz="10" samples="1800" gpu="${gpu}" >
     <origin xyz="0 0 ${base_z_size + 0.38}" rpy="0 0 0" />
-  </VLP-64>
+  </VLP-64> -->
+  <!-- Customized_LiDAR -->
+    <xacro:Customized_LiDAR parent="base_link" name="sensor" topic="Ruby80" gpu="true" ns="/">
+        <origin xyz="0 0 0.08" rpy="0 0 0" />
+    </xacro:Customized_LiDAR>
   <!-- rslidar-80 -->
   <!---->

Commit message: add velodyne OK

File: src/vehicle/mr1000/urdf/mr1000_motor.urdf.xacro (robot description, xacro)
@@ -38,6 +38,7 @@
   <xacro:include filename="$(find mr1000)/urdf/VLP-64.urdf.xacro"/>
   <!-- <xacro:include filename="$(find velodyne_description)/urdf/RS-Ruby80.urdf.xacro"/> -->
-  <xacro:include filename="$(find mr1000)/urdf/Customized.urdf.xacro"/>
+  <!-- <xacro:include filename="$(find mr1000)/urdf/Customized.urdf.xacro"/> -->
   <!-- <xacro:include filename="$(find velodyne_description)/urdf/VLP-16.urdf.xacro"/> -->
+  <xacro:include filename="$(find ouster_os1_64)/urdf/os1_64.urdf.xacro"/>
   <!-- Base link is the center of the robot's base -->
   <link name="base_link">
@@ -160,8 +161,12 @@
     <origin xyz="0 0 ${base_z_size + 0.38}" rpy="0 0 0" />
   </VLP-64> -->
+  <!-- os1_64 -->
+  <xacro:os1_64 parent="base" name="ouster" prefix="/os1_cloud_node" hz="10" samples="512"  gpu="true">
+    <origin xyz="0 0 1" rpy="0 0 0" />
+  </xacro:os1_64>
   <!-- Customized_LiDAR -->
-    <xacro:Customized_LiDAR parent="base_link" name="sensor" topic="Ruby80" gpu="true" ns="/">
+    <!-- <xacro:Customized_LiDAR parent="base_link" name="sensor" topic="Ruby80" gpu="true" ns="/">
         <origin xyz="0 0 0.08" rpy="0 0 0" />
-    </xacro:Customized_LiDAR>
+    </xacro:Customized_LiDAR> -->
   <!-- rslidar-80 -->
   <!---->
